Commit message: add light

File: src/ur_description/urdf/common.gazebo.xacro (robot description, xacro)
@@ -5,4 +5,13 @@
       <!--robotNamespace>/</robotNamespace-->
       <!--robotSimType>gazebo_ros_control/DefaultRobotHWSim</robotSimType-->
+    </plugin>
+    <plugin name="attach_light" filename="libAttachLightPlugin.so">
+      <link>
+        <link_name>wrist_3_link</link_name>
+        <light>
+          <pose>0 0 0 1.57 0 0</pose>
+          <light_name>spot</light_name>
+        </light>
+      </link>
     </plugin>
 <!--
